File: examples/tutorial-project/designs/gateway/gateway.kicad_sch (KiCad schematic)
At the start: 19 parts

Commit message: The tutorial board is a Sample Board
"ECU" is a private design name and it should not be in a public repo. It ran
through the tutorial fixture's titles, the project and review manifests, the
KiCad title blocks generated from them, four Go and TypeScript test fixtures,
three docsite pages, and every committed run capture that prints a manifest or a
sheet name.

The board keeps its `gateway` identifier everywhere. That is a slug, it is in
paths the tutorial types out, and renaming it would rewrite the ladder for no
confidentiality gain. Only the human-readable titles change.

Four sites used the term generically rather than as a name, describing industry
practice in a comment or a benchmark caption. Those are rewritten rather than
substituted, because the sentence wanted a plain noun and not another proper one.

Regenerated rather than hand-edited: the KiCad schematic and board come from
tools/gen_kicad_views.py and tools/gen_kicad_board.py, and re-running them
reproduces the committed files exactly, so the generators and their artifacts
still agree. The learn/ captures move by one line each, their #agni-run stamp,
which hashes the fixture. The fixture changed, so the stamp did.

docsite/static/designs/*.svg are NOT regenerated here. Running `make -C docsite
designs` picks up an unrelated renderer drift (font-family and every font-size),
which is a separate staleness worth its own diff. Only the title string is
substituted in gateway-schematic.svg, and gateway-netlist.svg never carried the
name.

This removes the term from the tree. It does not remove it from history, and the
history is public.
Other:
- title: Gateway ECU (tutorial board) -> Sample Board
Changed lines of the file:
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@@
 	(paper "A4")
 	(title_block
-		(title "Gateway ECU (tutorial board)")
+		(title "Sample Board")
 		(rev "A"))
 	(symbol (lib_id "gateway:CONN4") (at 25.4 25.4 0) (unit 1) (uuid "ij1")
